Commit message: Add rough urdf description of robot

File: description/robot.urdf.xacro (robot description, xacro)
@@ -2,4 +2,3 @@
 <robot xmlns:xacro="http://www.ros.org/wiki/xacro"  name="robot">
     <xacro:include filename="robot_core.xacro"/>
-    <xacro:include filename="colours.xacro"/>
 </robot>

File: description/robot_core.xacro (robot description, xacro)
@@ -1,14 +1,95 @@
 <?xml version="1.0"?>
 <robot xmlns:xacro="http://www.ros.org/wiki/xacro">
+    <xacro:include filename="colours.xacro"/>
+    <xacro:include filename="inertial_macros.xacro"/>
+    <xacro:property name="chassis_radius" value="0.07"/>
+    <xacro:property name="chassis_height" value="0.115"/>
+    <xacro:property name="wheel_radius" value="0.0325"/>
+    <xacro:property name="wheel_width" value="0.025"/>
+    <xacro:property name="caster_wheel_radius" value="0.0175"/>
+    <xacro:property name="wheel_offset" value="${chassis_radius-wheel_width/2+0.005}"/>
     <link name="base_link">
     </link>
     <link name="chassis">
         <visual>
-            <origin xyz="0 0 0.035" rpy="0 0 0"/>
+            <origin xyz="0 0 ${chassis_height/2}" rpy="0 0 0"/>
             <geometry>
-                <cylinder radius="${0.14/2}" length="${0.150-0.035}"/>
+                <cylinder radius="${chassis_radius}" length="${chassis_height}"/>
             </geometry>
             <material name="white"/>
         </visual>
+        <collision>
+            <origin xyz="0 0 ${chassis_height/2}" rpy="0 0 0"/>
+            <geometry>
+                <cylinder radius="${chassis_radius}" length="${chassis_height}"/>
+            </geometry>
+        </collision>
+        <xacro:inertial_cylinder mass="0.5" radius="${chassis_radius}" length="${chassis_height}">
+            <origin xyz="0 0 ${chassis_height/2}" rpy="0 0 0"/>
+        </xacro:inertial_cylinder>
+    </link>
+    <link name="left_wheel">
+        <visual>
+            <geometry>
+                <cylinder radius="${wheel_radius}" length="${wheel_width}"/>
+            </geometry>
+            <material name="blue"/>
+        </visual>
+        <collision>
+            <geometry>
+                <cylinder radius="${wheel_radius}" length="${wheel_width}"/>
+            </geometry>
+        </collision>
+        <xacro:inertial_cylinder mass="0.1" radius="${wheel_radius}" length="${wheel_width}">
+            <origin xyz="0 0 0" rpy="0 0 0"/>
+        </xacro:inertial_cylinder>
+    </link>
+    <link name="right_wheel">
+        <visual>
+            <geometry>
+                <cylinder radius="${wheel_radius}" length="${wheel_width}"/>
+            </geometry>
+            <material name="blue"/>
+        </visual>
+        <collision>
+            <geometry>
+                <cylinder radius="${wheel_radius}" length="${wheel_width}"/>
+            </geometry>
+        </collision>
+        <xacro:inertial_cylinder mass="0.1" radius="${wheel_radius}" length="${wheel_width}">
+            <origin xyz="0 0 0" rpy="0 0 0"/>
+        </xacro:inertial_cylinder>
+    </link>
+    <link name="top_caster_wheel">
+        <visual>
+            <geometry>
+                <sphere radius="${caster_wheel_radius}"/>
+            </geometry>
+            <material name="black"/>
+        </visual>
+        <collision>
+            <geometry>
+                <sphere radius="${caster_wheel_radius}"/>
+            </geometry>
+        </collision>
+        <xacro:inertial_sphere mass="0.1" radius="${caster_wheel_radius}">
+            <origin xyz="0 0 0" rpy="0 0 0"/>
+        </xacro:inertial_sphere>
+    </link>
+    <link name="bottom_caster_wheel">
+        <visual>
+            <geometry>
+                <sphere radius="${caster_wheel_radius}"/>
+            </geometry>
+            <material name="black"/>
+        </visual>
+        <collision>
+            <geometry>
+                <sphere radius="${caster_wheel_radius}"/>
+            </geometry>
+        </collision>
+        <xacro:inertial_sphere mass="0.1" radius="${caster_wheel_radius}">
+            <origin xyz="0 0 0" rpy="0 0 0"/>
+        </xacro:inertial_sphere>
     </link>
     <joint name="chassis_joint" type="fixed">
@@ -17,3 +98,25 @@
         <origin xyz="0 0 0"/>
     </joint>
+    <joint name="left_wheel_joint" type="continuous">
+        <parent link="base_link"/>
+        <child link="left_wheel"/>
+        <origin xyz="0 ${wheel_offset} 0" rpy="-${pi/2} 0 0"/>
+        <axis xyz="0 0 1"/>
+    </joint>
+    <joint name="right_wheel_joint" type="continuous">
+        <parent link="base_link"/>
+        <child link="right_wheel"/>
+        <origin xyz="0 -${wheel_offset} 0" rpy="${pi/2} 0 0"/>
+        <axis xyz="0 0 1"/>
+    </joint>
+    <joint name="top_caster_wheel_joint" type="fixed">
+        <parent link="chassis"/>
+        <child link="top_caster_wheel"/>
+        <origin xyz="0.05 0 -${0.035/2}" rpy="0 0 0"/>
+    </joint>
+    <joint name="bottom_caster_wheel_joint" type="fixed">
+        <parent link="chassis"/>
+        <child link="bottom_caster_wheel"/>
+        <origin xyz="-0.05 0 -${0.035/2}" rpy="0 0 0"/>
+    </joint>
 </robot>

Commit message: Get ros2 control sim setup working

File: description/robot.urdf.xacro (robot description, xacro)
@@ -3,3 +3,4 @@
     <xacro:include filename="robot_core.xacro"/>
     <xacro:include filename="ros2_control.xacro"/>
+    <!--xacro:include filename="gz.xacro"/-->
 </robot>

File: description/robot_core.xacro (robot description, xacro)
@@ -8,5 +8,6 @@
     <xacro:property name="wheel_width" value="0.025"/>
     <xacro:property name="caster_wheel_radius" value="0.0175"/>
-    <xacro:property name="wheel_offset" value="${chassis_radius-wheel_width/2+0.005}"/>
+    <xacro:property name="wheel_offset" value="${chassis_radius+0.015}"/>
+    <!--xacro:property name="wheel_offset" value="${chassis_radius-wheel_width/2+0.005}"/-->
     <link name="base_link">
     </link>
@@ -66,5 +67,5 @@
                 <sphere radius="${caster_wheel_radius}"/>
             </geometry>
-            <material name="black"/>
+            <material name="orange"/>
         </visual>
         <collision>
@@ -108,15 +109,23 @@
         <child link="right_wheel"/>
         <origin xyz="0 -${wheel_offset} 0" rpy="${pi/2} 0 0"/>
-        <axis xyz="0 0 1"/>
+        <axis xyz="0 0 -1"/>
     </joint>
     <joint name="top_caster_wheel_joint" type="fixed">
         <parent link="chassis"/>
         <child link="top_caster_wheel"/>
-        <origin xyz="0.05 0 -${0.035/2}" rpy="0 0 0"/>
+        <origin xyz="0.05 0 -0.015" rpy="0 0 0"/>
     </joint>
     <joint name="bottom_caster_wheel_joint" type="fixed">
         <parent link="chassis"/>
         <child link="bottom_caster_wheel"/>
-        <origin xyz="-0.05 0 -${0.035/2}" rpy="0 0 0"/>
+        <origin xyz="-0.05 0 -0.015" rpy="0 0 0"/>
     </joint>
+    <gazebo reference="top_caster_wheel">
+        <mu1 value="0.001"/>
+        <mu2 value="0.001"/>
+    </gazebo>
+    <gazebo reference="bottom_caster_wheel">
+        <mu1 value="0.001"/>
+        <mu2 value="0.001"/>
+    </gazebo>
 </robot>

File: description/ros2_control.xacro (robot description, xacro)
@@ -24,4 +24,6 @@
     <gazebo>
         <plugin filename="ign_ros2_control-system" name="ign_ros2_control::IgnitionROS2ControlPlugin">
+            <robot_param>robot_description</robot_param>
+            <robot_param_node>robot_state_publisher</robot_param_node>
             <parameters>$(find ros2_dd_robot)/config/my_controllers.yaml</parameters>
         </plugin>

Commit message: Switched to spherical collisions for wheels

File: description/robot.urdf.xacro (robot description, xacro)
@@ -3,4 +3,3 @@
     <xacro:include filename="robot_core.xacro"/>
     <xacro:include filename="ros2_control.xacro"/>
-    <!--xacro:include filename="gz.xacro"/-->
 </robot>

File: description/robot_core.xacro (robot description, xacro)
@@ -38,6 +38,11 @@
         </visual>
         <collision>
+            <!--
             <geometry>
                 <cylinder radius="${wheel_radius}" length="${wheel_width}"/>
+            </geometry>
+            -->
+            <geometry>
+                <sphere radius="${wheel_radius}"/>
             </geometry>
         </collision>
@@ -54,6 +59,11 @@
         </visual>
         <collision>
+            <!--
             <geometry>
                 <cylinder radius="${wheel_radius}" length="${wheel_width}"/>
+            </geometry>
+            -->
+            <geometry>
+                <sphere radius="${wheel_radius}"/>
             </geometry>
         </collision>
